File: Signal_Generator_PCB/Signal_Generator_PCB.kicad_sch (KiCad schematic)
At the start: 0 parts

Commit message: feat:(develop) Añado la primer versión del esquemático y PCB
Parts:
- added J1: Conn_01x04, DM-OLED096-636:MODULE_DM-OLED096-636, symbol Connector_Generic:Conn_01x04
- added J2: Conn_01x02, Connector_PinHeader_2.54mm:PinHeader_1x02_P2.54mm_Vertical, symbol Connector_Generic:Conn_01x02
- added R1, R2, R3: 10k, Resistor_THT:R_Axial_DIN0207_L6.3mm_D2.5mm_P10.16mm_Horizontal, symbol Device:R
- added SW1: RotaryEncoder_Switch, Rotary_Encoder:RotaryEncoder_Alps_EC11E-Switch_Vertical_H20mm_MountingHoles, symbol Device:RotaryEncoder_Switch
- added U1: ESP32-DevKitC, PCM_Espressif:ESP32-DevKitC, symbol PCM_Espressif:ESP32-DevKitC
Connections:
- new net +3.3V: J1.2 (VDD), R1.2, R2.2, R3.2, U1.1 (3V3)
- new net GNDREF: J1.1 (GND), J2.1 (Pin_1), SW1.C, SW1.S2, U1.14 (GND), U1.32 (GND), U1.38 (GND)
- new net GPIO12: R3.1, SW1.S1, U1.13 (MTDI/GPIO12/ADC2_CH5)
- new net GPIO14: R1.1, SW1.B, U1.12 (MTMS/GPIO14/ADC2_CH6)
- new net GPIO21: J1.4 (SDA), U1.33 (GPIO21)
- new net GPIO22: J1.3 (SCK), U1.36 (GPIO22)
- new net GPIO25: J2.2 (Pin_2), U1.9 (DAC_1/ADC2_CH8/GPIO25)
- new net GPIO27: R2.1, SW1.A, U1.11 (ADC2_CH7/GPIO27)
- no-connect marks 0 -> 26
Other:
- note added: "CLK"
- note added: "DT"
- note added: "ESP32-WROOM"
- note added: "Encoder Rotativo con Switch"
- note added: "Output"
- note added: "Pantalla OLED"
- note added: "SW"

Commit message: feat(Signal_Generator): Añado los header files.
Connections:
- no-connect marks 26 -> 27
Changed lines of the file:
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@@
+	)
+	(no_connect
+		(at 64.77 27.94)
 	)
 	(no_connect

Commit message: feat(Signal_Generator_PCB): v02
Parts:
- added J3: Conn_01x02, symbol Connector_Generic:Conn_01x02
Connections:
- net GPIO25: now also J2.1 (Pin_1); no longer J2.2 (Pin_2)
- net +5V: now reaches U1.19 (5V)
- net +5V: now also J3.2 (Pin_2)
- net GNDREF renamed GND
- net GND: now also J2.2 (Pin_2), J3.1 (Pin_1); no longer J2.1 (Pin_1)
- no-connect marks 27 -> 26
Other:
- note added: "+5V from USB-C via external source"
- note added: "OLED Screen"
- note added: "Rotary Encoder with Switch"
- note removed: "Encoder Rotativo con Switch"
- note removed: "Pantalla OLED"
- moved on the sheet: J1, J2, R1, R2, R3, SW1, U1

Commit message: feat(PCB): Cambios en la configuración de la PCB.
Connections:
- net GPIO32: now reaches U1.7 (32K_XP/GPIO32/ADC1_CH4)
- net GPIO32: now also R3.1, SW1.S1
- removed net GPIO12: R3.1, SW1.S1, U1.13 (MTDI/GPIO12/ADC2_CH5)
- no-connect marks 26 -> 27
Other:
- note added: "SCL"
- note added: "SDA"
Changed lines of the file:
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@@
 		(title "ESP32 SIgnal Generator")
 		(date "2026-09")
-		(rev "v02")
+		(rev "v03")
 		(company "UTNFRA")
 		(comment 1 "Alvarez Mollo, Fausto")
@@
 		)
 	)
+	(text "SDA"
+		(exclude_from_sim no)
+		(at 127.254 70.358 0)
+		(effects
+			(font
+				(size 1.27 1.27)
+			)
+		)
+	)
 	(text "CLK"
 		(exclude_from_sim no)
@@
 		(exclude_from_sim no)
 		(at 95.504 105.156 0)
+		(effects
+			(font
+				(size 1.27 1.27)
+			)
+		)
+	)
+	(text "SCL"
+		(exclude_from_sim no)
+		(at 127.254 72.898 0)
 		(effects
 			(font
@@
 	)
 	(no_connect
+		(at 92.71 91.44)
+	)
+	(no_connect
 		(at 26.67 63.5)
 	)
@@
 	)
 	(no_connect
+		(at 92.71 63.5)
+	)
+	(no_connect
 		(at 92.71 78.74)
 	)
@@
 	)
 	(no_connect
-		(at 92.71 63.5)
-	)
-	(no_connect
-		(at 26.67 35.56)
-	)
-	(no_connect
 		(at 26.67 55.88)
 	)
@@
 	)
 	(no_connect
+		(at 26.67 43.18)
+	)
+	(no_connect
 		(at 92.71 73.66)
 	)
@@
 	(wire
 		(pts
+			(xy 24.13 35.56) (xy 26.67 35.56)
+		)
+		(stroke
+			(width 0)
+			(type default)
+		)
+	)
+	(wire
+		(pts
 			(xy 132.08 54.61) (xy 128.27 54.61)
 		)
@@
 		(pts
 			(xy 144.78 92.71) (xy 142.24 92.71)
-		)
-		(stroke
-			(width 0)
-			(type default)
-		)
-	)
-	(wire
-		(pts
-			(xy 24.13 43.18) (xy 26.67 43.18)
 		)
 		(stroke
@@
 		)
 	)
-	(label "GPIO12"
+	(label "GPIO32"
 		(at 149.86 36.83 0)
 		(fields_autoplaced yes)
@@
 		)
 	)
-	(label "GPIO12"
-		(at 24.13 43.18 180)
+	(label "GPIO32"
+		(at 24.13 35.56 180)
 		(fields_autoplaced yes)
 		(effects
@@
 		)
 		(property "GPIO" ""
-			(at 24.13 44.45 0)
-			(show_name no)
-			(do_not_autoplace no)
+			(at 24.13 36.83 0)
+			(show_name no)
+			(do_not_autoplace no)
